Commit message: Modify entire codes (todo: diagonal)

File: tr_dual_steering/robots/tr_robot.xacro (robot description, xacro)
@@ -17,20 +17,20 @@
     <xacro:property name="caster_b_half" value="${p['caster_b_half']}"/>
     <!-- base -->
-    <link name="base_link" />
+    <link name="base_footprint" />
     <xacro:dual_steering_robot_base
-      name="base_footprint"
-      parent="base_link">
+      name="base_link"
+      parent="base_footprint">
       <origin xyz="0 0 0" rpy="0 0 0" />
     </xacro:dual_steering_robot_base>
     <!-- front qd wheel -->
     <xacro:qd_wheel_160
-      name="robot_qd_wheel_${front_name}"
-      parent="base_footprint">
+      name="${front_name}"
+      parent="base_link">
       <origin xyz="${L_half} ${-B_half} ${-qd_height}" rpy="0 0 0" />
     </xacro:qd_wheel_160>
     <!-- rear qd wheel -->
     <xacro:qd_wheel_160
-      name="robot_qd_wheel_${rear_name}"
-      parent="base_footprint">
+      name="${rear_name}"
+      parent="base_link">
       <origin xyz="${-L_half} ${B_half} ${-qd_height}" rpy="0 0 0" />
     </xacro:qd_wheel_160>
@@ -38,5 +38,5 @@
     <xacro:caster_wheel_75
       name="robot_caster_wheel_front_left"
-      parent="base_footprint">
+      parent="base_link">
       <origin xyz="${L_half} ${caster_b_half} ${-caster_height}" rpy="0 0 0" />
     </xacro:caster_wheel_75>
@@ -44,5 +44,5 @@
     <xacro:caster_wheel_75
       name="robot_caster_wheel_rear_right"
-      parent="base_footprint">
+      parent="base_link">
       <origin xyz="${-L_half} ${-caster_b_half} ${-caster_height}" rpy="0 0 0"/>
     </xacro:caster_wheel_75>
@@ -52,5 +52,5 @@
       <xacro:caster_wheel_75
         name="robot_caster_wheel_front_right"
-        parent="base_footprint">
+        parent="base_link">
         <origin xyz="${L_half} ${-caster_b_half}  ${-caster_height}" rpy="0 0 0" />
       </xacro:caster_wheel_75>
@@ -58,8 +58,9 @@
       <xacro:caster_wheel_75
         name="robot_caster_wheel_rear_left"
-        parent="base_footprint">
+        parent="base_link">
         <origin xyz="${-L_half} ${caster_b_half}  ${-caster_height}" rpy="0 0 0" />
       </xacro:caster_wheel_75>
     </xacro:if>
+    <xacro:include filename="$(find tr_dual_steering)/robots/xacros/gazebo.urdf.xacro"/>
   </xacro:macro>
 </robot>

File: tr_dual_steering/robots/xacros/caster_wheel.xacro (robot description, xacro)
@@ -1,17 +1,16 @@
 <?xml version="1.0"?>
 <robot xmlns:xacro="http://www.ros.org/wiki/xacro" name="dual_steering_robot">
-  <xacro:macro name="caster_wheel_75" params="name parent *origin">
-   <joint name="${name}_mount_joint" type="revolute">
+  <xacro:macro name="caster_wheel_75"
+               params="name parent *origin
+                       frictionless:=true mu1:=0.0 mu2:=0.0 slip1:=1.0 slip2:=1.0">
+   <joint name="${name}_mount_joint" type="continuous">
     <xacro:insert_block name="origin" />
-    <axis xyz="0 0 -1" />
-    <joint_properties damping="100" friction="1000" />
-        <limit effort="1000.0" lower="-1e+16" upper="1e+16" velocity="1.02"/>
-    <joint_properties damping="1.0" friction="1" />
-    <dynamics damping="1.0" friction="1" />
-    <limit effort="1000.0" lower="-1e+16" upper="1e+16" velocity="1.02"/>
+    <axis xyz="0 0 1" />
+    <dynamics damping="0.2" />
+    <!-- <limit effort="1000.0" lower="-3.14" upper="3.14" velocity="1.02"/> -->
     <parent link="${parent}" />
     <child link="${name}_mount_link" />
    </joint>
-   <link name="${name}_mount_link" type="wheel">
+   <link name="${name}_mount_link">
     <inertial>
       <mass value="2.2" />
@@ -28,25 +27,21 @@
     </visual>
     <collision>
-     <origin xyz="0 0 0" rpy="0 1.57 1.57" />
+     <origin xyz="0 0 0" rpy="0 0 0" />
      <geometry>
-       <!-- <cylinder radius="0.075" length="0.046"/> -->
-      <sphere radius="0.075" />
+        <cylinder radius="0.075" length="0.22"/>
      </geometry>
     </collision>
    </link>
-   <joint name="${name}_joint" type="revolute">
-    <origin xyz="0 0 -0.185" rpy="1.571 0 0" />
+   <joint name="${name}_joint" type="continuous">
+    <origin xyz="0 0 -0.185" rpy="-1.57 0 0" />
     <axis xyz="0 0 1" />
-    <joint_properties damping="100" friction="1000" />
-        <limit effort="1000.0" lower="-1e+16" upper="1e+16" velocity="1.02"/>
-    <joint_properties damping="1.0" friction="1" />
-    <!-- <dynamics damping="1.0" friction="1" />
-    <limit effort="1000.0" lower="-1e+16" upper="1e+16" velocity="1.02"/> -->
+    <dynamics damping="0.01" />
+    <!-- <limit effort="1000.0" lower="-3.14" upper="3.14" velocity="1.02"/> -->
     <parent link="${name}_mount_link" />
     <child link="${name}_link" />
    </joint>
-   <link name="${name}_link" type="wheel">
+   <link name="${name}_link">
     <inertial>
-      <mass value="2.2" />
+      <mass value="8" />
       <origin xyz="0 0 0" rpy="0 0 0" />
         <inertia  ixx="0.01" ixy="0.0" ixz="0.0"
@@ -61,18 +56,20 @@
     </visual>
     <collision>
-     <origin xyz="0 0 0" rpy="0 1.57 1.57" />
+     <origin xyz="0 0 0" rpy="0 0 0" />
      <geometry>
-       <!-- <cylinder radius="0.075" length="0.046"/> -->
-      <sphere radius="0.075" />
+        <cylinder radius="0.075" length="0.046"/>
      </geometry>
     </collision>
    </link>
-<gazebo reference="${name}_link">
-      <!-- <kp> 10000 </kp> -->
-      <!-- <fdir1>0 1 0</fdir1> -->
-      <!-- <slip1> 0.1 </slip1> -->
-      <mu1>0.0001</mu1>
-      <mu2>0.0001</mu2>
-</gazebo>
+   <xacro:if value="${frictionless}">
+      <gazebo reference="${name}_link">
+         <mu1>${mu1}</mu1><mu2>${mu2}</mu2>
+         <slip1>${slip1}</slip1><slip2>${slip2}</slip2>
+      </gazebo>
+      <gazebo reference="${name}_mount_link">
+         <mu1>${mu1}</mu1><mu2>${mu2}</mu2>
+         <slip1>${slip1}</slip1><slip2>${slip2}</slip2>
+      </gazebo>
+   </xacro:if>
   </xacro:macro>
 </robot>

File: tr_dual_steering/robots/xacros/dual_steering_robot_body.xacro (robot description, xacro)
@@ -2,22 +2,14 @@
 <robot xmlns:xacro="http://www.ros.org/wiki/xacro" name="dual_steering_robot">
   <xacro:macro name="dual_steering_robot_base" params="name parent *origin">
-    <joint name="${name}_joint" type="fixed">
-      <xacro:insert_block name="origin" />
-      <axis xyz="0 0 -1" />
-      <!-- <limit effort="1000.0" lower="-1e+16" upper="1e+16" velocity="3.5"/> -->
-      <joint_properties damping="1" friction="1" />
-      <parent link="${parent}" />
-      <child link="${name}" />
-   </joint>
     <link name="${name}">
       <inertial>
-        <mass value="64"/>
-        <origin xyz="0 0.0 0.0" />
+        <mass value="55"/>
+        <origin xyz="0.0 0.0 0.0" />
          <inertia ixx="2.8" ixy="0.0" ixz="0.0"
-                 iyy="2.8" iyz="0.0"
-                 izz="2.8" />
+                  iyy="2.8" iyz="0.0"
+                  izz="2.8" />
       </inertial>
       <visual>
-        <origin xyz="0. 0. 0" rpy="0 0 0" />
+        <origin xyz="0.0 0.0 0.0" rpy="0 0 0" />
         <geometry>
             <box size="1.4 1.0 0.24"/>
@@ -25,5 +17,5 @@
       </visual>
       <collision>
-        <origin xyz="0. 0. 0.0" rpy="-1.571 0 1.571" />
+        <origin xyz="0.0 0.0 0.0" rpy="0 0 0" />
         <geometry>
             <box size="1.0 0.80 0.24"/>
@@ -31,4 +23,9 @@
       </collision>
     </link>
+    <joint name="${name}_joint" type="fixed">
+      <xacro:insert_block name="origin" />
+      <parent link="${parent}" />
+      <child link="${name}" />
+   </joint>
   </xacro:macro>
 </robot>

File: tr_dual_steering/robots/xacros/qd_wheel.xacro (robot description, xacro)
@@ -2,15 +2,15 @@
 <robot xmlns:xacro="http://www.ros.org/wiki/xacro" name="dual_steering_robot">
   <xacro:macro name="qd_wheel_160" params="name parent *origin">
-   <joint name="${name}_steer_joint" type="revolute">
+   <joint name="${name}_steer_joint" type="continuous">
     <xacro:insert_block name="origin" />
-    <axis xyz="0 0 -1" />
-    <dynamics damping="1.0" friction="1" />
-    <limit effort="1000.0" lower="-1e+16" upper="1e+16" velocity="1.02"/>
+    <axis xyz="0 0 1" />
+    <dynamics damping="0.2" />
+    <!-- <limit effort="1000.0" lower="-1.57" upper="1.57" velocity="1.02"/> -->
     <parent link="${parent}" />
     <child link="${name}_steer_link" />
    </joint>
-   <link name="${name}_steer_link" type="wheel">
+   <link name="${name}_steer_link">
     <inertial>
-      <mass value="2.2" />
+      <mass value="1" />
       <origin xyz="0 0 0" rpy="0 0 0" />
         <inertia  ixx="0.01" ixy="0.0" ixz="0.0"
@@ -25,23 +25,21 @@
     </visual>
     <collision>
-     <origin xyz="0 0 0" rpy="0 1.571 1.571" />
+     <origin xyz="0 0 0" rpy="0 0 0" />
      <geometry>
-       <!-- <cylinder radius="0.16" length="0.05"/> -->
-      <sphere radius="0.16" />
+        <cylinder radius="0.16" length="0.05"/>
      </geometry>
     </collision>
    </link>
-   <joint name="${name}_drive_joint" type="revolute">
-    <origin xyz="0 0 -0.185" rpy="1.571 0 0" />
+   <joint name="${name}_drive_joint" type="continuous">
+    <origin xyz="0 0 -0.185" rpy="-1.57 0 0" />
     <axis xyz="0 0 1" />
-    <joint_properties damping="100" friction="1000" />
-        <limit effort="1000.0" lower="-1e+16" upper="1e+16" velocity="1.02"/>
-    <joint_properties damping="1.0" friction="1" />
+    <dynamics damping="0.01" />
+    <!-- <limit effort="1000.0" lower="-3.14" upper="3.14" velocity="1.02"/> -->
     <parent link="${name}_steer_link" />
     <child link="${name}_drive_link" />
    </joint>
-   <link name="${name}_drive_link" type="wheel">
+   <link name="${name}_drive_link">
     <inertial>
-      <mass value="2.2" />
+      <mass value="8.0" />
       <origin xyz="0 0 0" rpy="0 0 0" />
         <inertia  ixx="0.01" ixy="0.0" ixz="0.0"
@@ -56,18 +54,10 @@
     </visual>
     <collision>
-     <origin xyz="0 0 0" rpy="0 1.571 1.571" />
+     <origin xyz="0 0 0" rpy="0 0 0" />
      <geometry>
-       <!-- <cylinder radius="0.16" length="0.05"/> -->
-      <sphere radius="0.16" />
+        <cylinder radius="0.16" length="0.05"/>
      </geometry>
     </collision>
    </link>
-<gazebo reference="${name}_link">
-      <!-- <kp> 10000 </kp> -->
-      <!-- <fdir1>0 1 0</fdir1> -->
-      <!-- <slip1> 0.1 </slip1> -->
-      <mu1>0.0001</mu1>
-      <mu2>0.0001</mu2>
-</gazebo>
   </xacro:macro>
 </robot>

Commit message: Fix controller issues

File: tr_dual_steering/robots/tr_robot.xacro (robot description, xacro)
@@ -7,5 +7,5 @@
     <xacro:include filename="$(find tr_dual_steering)/robots/xacros/caster_wheel.xacro"/>
     <xacro:property name="cfg_name" value="${xacro.load_yaml(yaml_path)}"/>
-    <xacro:property name="p" value="${cfg_name['tr_dual_steering']['ros__parameters']}"/>
+    <xacro:property name="p" value="${cfg_name['tr_dual_steering_node']['ros__parameters']}"/>
     <xacro:property name="wheel_type" value="${p['wheel_type']}"/>
     <xacro:property name="front_name"    value="${p['module_names'][0]}"/>
@@ -27,5 +27,5 @@
       name="${front_name}"
       parent="base_link">
-      <origin xyz="${L_half} ${-B_half} ${-qd_height}" rpy="0 0 0" />
+      <origin xyz="${L_half} ${B_half} ${-qd_height}" rpy="0 0 0" />
     </xacro:qd_wheel_160>
     <!-- rear qd wheel -->
@@ -33,5 +33,5 @@
       name="${rear_name}"
       parent="base_link">
-      <origin xyz="${-L_half} ${B_half} ${-qd_height}" rpy="0 0 0" />
+      <origin xyz="${-L_half} ${-B_half} ${-qd_height}" rpy="0 0 0" />
     </xacro:qd_wheel_160>
     <!-- front left caster wheel -->
@@ -39,5 +39,5 @@
       name="robot_caster_wheel_front_left"
       parent="base_link">
-      <origin xyz="${L_half} ${caster_b_half} ${-caster_height}" rpy="0 0 0" />
+      <origin xyz="${L_half} ${-caster_b_half} ${-caster_height}" rpy="0 0 0" />
     </xacro:caster_wheel_75>
     <!-- rear right caster wheel -->
@@ -45,5 +45,5 @@
       name="robot_caster_wheel_rear_right"
       parent="base_link">
-      <origin xyz="${-L_half} ${-caster_b_half} ${-caster_height}" rpy="0 0 0"/>
+      <origin xyz="${-L_half} ${caster_b_half} ${-caster_height}" rpy="0 0 0"/>
     </xacro:caster_wheel_75>
     <!-- caster wheel for aligned type -->
@@ -53,5 +53,5 @@
         name="robot_caster_wheel_front_right"
         parent="base_link">
-        <origin xyz="${L_half} ${-caster_b_half}  ${-caster_height}" rpy="0 0 0" />
+        <origin xyz="${L_half} ${caster_b_half}  ${-caster_height}" rpy="0 0 0" />
       </xacro:caster_wheel_75>
       <!-- rear left caster wheel -->
@@ -59,5 +59,5 @@
         name="robot_caster_wheel_rear_left"
         parent="base_link">
-        <origin xyz="${-L_half} ${caster_b_half}  ${-caster_height}" rpy="0 0 0" />
+        <origin xyz="${-L_half} ${-caster_b_half}  ${-caster_height}" rpy="0 0 0" />
       </xacro:caster_wheel_75>
     </xacro:if>

Commit message: Add Kinematics & SLAM & Navigation

File: tr_dual_steering/robots/tr_robot.xacro (robot description, xacro)
@@ -4,6 +4,6 @@
                params="yaml_path">
     <xacro:include filename="$(find tr_dual_steering)/robots/xacros/dual_steering_robot_body.xacro"/>
-    <xacro:include filename="$(find tr_dual_steering)/robots/xacros/qd_wheel.xacro"/>
-    <xacro:include filename="$(find tr_dual_steering)/robots/xacros/caster_wheel.xacro"/>
+    <xacro:include filename="$(find tr_dual_steering)/robots/xacros/wheel/qd_wheel.xacro"/>
+    <xacro:include filename="$(find tr_dual_steering)/robots/xacros/wheel/caster_wheel.xacro"/>
     <xacro:property name="cfg_name" value="${xacro.load_yaml(yaml_path)}"/>
     <xacro:property name="p" value="${cfg_name['tr_dual_steering_node']['ros__parameters']}"/>
@@ -21,5 +21,5 @@
       name="base_link"
       parent="base_footprint">
-      <origin xyz="0 0 0" rpy="0 0 0" />
+      <origin xyz="0 0 0.49" rpy="0 0 0" />
     </xacro:dual_steering_robot_base>
     <!-- front qd wheel -->
@@ -62,5 +62,5 @@
       </xacro:caster_wheel_75>
     </xacro:if>
-    <xacro:include filename="$(find tr_dual_steering)/robots/xacros/gazebo.urdf.xacro"/>
+    <xacro:include filename="$(find tr_dual_steering)/robots/gazebo.urdf.xacro"/>
   </xacro:macro>
 </robot>

File: tr_dual_steering/robots/xacros/dual_steering_robot_body.xacro (robot description, xacro)
@@ -10,14 +10,14 @@
                   izz="2.8" />
       </inertial>
-      <visual>
+      <!-- <visual>
         <origin xyz="0.0 0.0 0.0" rpy="0 0 0" />
         <geometry>
             <box size="1.4 1.0 0.24"/>
         </geometry>
-      </visual>
+      </visual> -->
       <collision>
         <origin xyz="0.0 0.0 0.0" rpy="0 0 0" />
         <geometry>
-            <box size="1.0 0.80 0.24"/>
+            <box size="1.4 1.0 0.24"/>
         </geometry>
       </collision>
