Commit message: add FAST_LIO_LOCALIZATION

File: tr_dual_steering/robots/gazebo.urdf.xacro (robot description, xacro)
@@ -3,10 +3,10 @@
   <xacro:include filename="$(find tr_dual_steering)/robots/xacros/VLP-16.urdf.xacro"/>
   <xacro:include filename="$(find tr_dual_steering)/robots/xacros/HDL-32E.urdf.xacro"/>
-  <xacro:VLP-16>
+  <!-- <xacro:VLP-16>
     <origin xyz="0 0 0.2305" rpy="0 0 0"/>
-  </xacro:VLP-16>
-  <!-- <xacro:HDL-32E>
-    <origin xyz="0 0 0.2332" rpy="0 0 0"/>
-  </xacro:HDL-32E> -->
+  </xacro:VLP-16> -->
+  <xacro:HDL-32E>
+    <origin xyz="0 0 0.2305" rpy="0 0 0"/>
+  </xacro:HDL-32E>
   <link name="imu_link">
     <inertial>
@@ -27,5 +27,5 @@
     <parent link="base_link"/>
     <child link="imu_link"/>
-    <origin xyz="0.1 0 0.12" rpy="0 0 0"/>
+    <origin xyz="0.0 0 0.12" rpy="0 0 0"/>
   </joint>
   <gazebo reference="imu_link">

File: tr_dual_steering/robots/xacros/HDL-32E.urdf.xacro (robot description, xacro)
@@ -54,5 +54,5 @@
     <gazebo reference="${name}">
       <xacro:if value="${gpu}">
-        <sensor type="gpu_ray" name="${name}-HDL32E">
+        <sensor type="gpu_ray" name="hdl32e">
           <pose>0 0 0 0 0 0</pose>
           <visualize>false</visualize>

File: tr_dual_steering/robots/xacros/VLP-16.urdf.xacro (robot description, xacro)
@@ -59,5 +59,5 @@
     <gazebo reference="${name}">
       <xacro:if value="${gpu}">
-        <sensor type="gpu_ray" name="${name}-VLP16">
+        <sensor type="gpu_ray" name="vlp16">
           <pose>0 0 0 0 0 0</pose>
           <visualize>false</visualize>

File: tr_dual_steering/robots/xacros/caster_wheel.xacro (robot description, xacro)
@@ -66,8 +66,10 @@
          <mu1>${mu1}</mu1><mu2>${mu2}</mu2>
          <slip1>${slip1}</slip1><slip2>${slip2}</slip2>
+         <material>Gazebo/Red</material>  <!-- Gazebo/Red, Gazebo/Green 등 -->
       </gazebo>
       <gazebo reference="${name}_mount_link">
          <mu1>${mu1}</mu1><mu2>${mu2}</mu2>
          <slip1>${slip1}</slip1><slip2>${slip2}</slip2>
+         <material>Gazebo/Red</material>  <!-- Gazebo/Red, Gazebo/Green 등 -->
       </gazebo>
    </xacro:if>

File: tr_dual_steering/robots/xacros/qd_wheel.xacro (robot description, xacro)
@@ -6,5 +6,5 @@
     <axis xyz="0 0 1" />
     <dynamics damping="0.3" />
-    <!-- <limit effort="1000.0" lower="-1.57" upper="1.57" velocity="1.02"/> -->
+    <limit effort="1000.0" lower="-1.57" upper="1.57" velocity="1.02"/>
     <parent link="${parent}" />
     <child link="${name}_steer_link" />
@@ -35,5 +35,5 @@
     <axis xyz="0 0 1" />
     <dynamics damping="0.015" />
-    <!-- <limit effort="1000.0" lower="-3.14" upper="3.14" velocity="1.02"/> -->
+    <limit effort="1000.0" velocity="1.02"/>
     <parent link="${name}_steer_link" />
     <child link="${name}_drive_link" />
@@ -60,4 +60,7 @@
     </collision>
    </link>
+   <gazebo reference="${name}_steer_link">
+      <material>Gazebo/Red</material>  <!-- Gazebo/Red, Gazebo/Green 등 -->
+   </gazebo>
    <gazebo reference="${name}_drive_link">
       <mu1>1.5</mu1>   <!-- 진행 방향 -->
@@ -65,4 +68,5 @@
       <slip1>0.01</slip1>
       <slip2>0.01</slip2>
+      <material>Gazebo/Red</material>  <!-- Gazebo/Red, Gazebo/Green 등 -->
    </gazebo>
   </xacro:macro>
